File: hardware/pcb/kxusbc2.kicad_sch (KiCad schematic)
At the start: 7 parts, among them J1 Conn_01x03, J3 Conn_01x03, J4 Conn_01x03, J7 Conn_01x01, J8 Conn_01x01

Commit message: Add bottom solder pads for mounting standoffs (closes #14)
Parts:
- H1, H2: footprint Mounting_Wuerth:Mounting_Wuerth_WA-SMSI-M2.5_H3mm_9774030151 -> Wuerth_9774030151_HS:Wuerth_9774030151_HS
Changed lines of the file:
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@@
 			)
 		)
-		(property "Footprint" "Mounting_Wuerth:Mounting_Wuerth_WA-SMSI-M2.5_H3mm_9774030151"
+		(property "Footprint" "Wuerth_9774030151_HS:Wuerth_9774030151_HS"
 			(at 53.34 170.18 0)
 			(effects
@@
 			)
 		)
-		(property "Datasheet" "~"
+		(property "Datasheet" ""
 			(at 53.34 170.18 0)
 			(effects
@@
 			)
 		)
-		(property "Description" "Mounting Hole with connection"
+		(property "Description" "with solder pad on bottom for hand soldering"
 			(at 53.34 170.18 0)
 			(effects
@@
 			)
 		)
-		(property "Footprint" "Mounting_Wuerth:Mounting_Wuerth_WA-SMSI-M2.5_H3mm_9774030151"
+		(property "Footprint" "Wuerth_9774030151_HS:Wuerth_9774030151_HS"
 			(at 60.96 170.18 0)
 			(effects
@@
 			)
 		)
-		(property "Datasheet" "~"
+		(property "Datasheet" ""
 			(at 60.96 170.18 0)
 			(effects
@@
 			)
 		)
-		(property "Description" "Mounting Hole with connection"
+		(property "Description" "with solder pad on bottom for hand soldering"
 			(at 60.96 170.18 0)
 			(effects
